File: security-system-pcb/security-system-schematic/security-system.kicad_pcb (KiCad board)
At the start: 4 copper layers, 102 x 41 mm, 11 parts, among them J1 Conn_01x06_Pin, J2 USB_C, U1 ESP32-Header

Commit message: Push changes to case and gerbers v1.4
Other:
- copper layers 4 -> 2
- board text added: "DECEMBER/26/2025 - v1.4"
- board text removed: "DECEMBER/26/2025 - v1.3"
Changed lines of the file:
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@@
 	(layers
 		(0 "F.Cu" signal "Front")
-		(4 "In1.Cu" signal)
-		(6 "In2.Cu" signal)
 		(2 "B.Cu" signal "Back")
 		(13 "F.Paste" user)
@@
 			(layer "dielectric 1"
 				(type "core")
-				(thickness 0.480066)
-				(material "FR4")
-				(epsilon_r 4.5)
-				(loss_tangent 0.02)
-			)
-			(layer "In1.Cu"
-				(type "copper")
-				(thickness 0.035)
-			)
-			(layer "dielectric 2"
-				(type "prepreg")
-				(thickness 0.480066)
-				(material "FR4")
-				(epsilon_r 4.5)
-				(loss_tangent 0.02)
-			)
-			(layer "In2.Cu"
-				(type "copper")
-				(thickness 0.035)
-			)
-			(layer "dielectric 3"
-				(type "core")
-				(thickness 0.480066)
+				(thickness 1.510198)
 				(material "FR4")
 				(epsilon_r 4.5)
@@
 			(drillshape 0)
 			(scaleselection 1)
-			(outputdirectory "gerbers/security-system-v1.3/")
+			(outputdirectory "gerbers/security-system-v1.4/")
 		)
 	)
@@
 		)
 	)
-	(gr_text "DECEMBER/26/2025 - v1.3"
+	(gr_text "DECEMBER/26/2025 - v1.4"
 		(at 153.012311 104.93 0)
 		(layer "F.SilkS")
